Commit message: working base

File: src/minolo/urdf/robot.urdf (robot description, URDF)
Before this commit: robot diglobot2, 5 links, 4 joints
Links:
- removed link base_link
- removed link scanner
- added link base_footprint; visual box size=0.48 0.3 0.01
- added link scanner_link; visual cylinder length=0.02 radius=0.025
Joints:
- joint base_to_fwheel: parent base_link -> base_footprint
- joint base_to_lwheel: parent base_link -> base_footprint
- joint base_to_rwheel: parent base_link -> base_footprint
- joint base_to_scanner: child scanner -> scanner_link; parent base_link -> base_footprint

Commit message: functioning_interface

File: src/minolo/urdf/robot.urdf (robot description, URDF)
Before this commit: robot diglobot2, 5 links, 4 joints
Joints:
- joint base_to_scanner: origin xyz=0.045 0 0.225 rpy=0 0 0 -> xyz=0.045 0 0.225 rpy=0 0 -1.57079

Commit message: fix IMU+odometry fusion

File: src/minolo/urdf/robot.urdf (robot description, URDF)
Before this commit: robot diglobot2, 5 links, 4 joints
Links:
- added link imu_link; visual box size=0.05 0.05 0.05
Joints:
- added joint imu_joint: type fixed, parent base_footprint, child imu_link, origin xyz=0.21 -0.02 0.15 rpy=0 0 0

Commit message: adding gps nav

File: src/minolo/urdf/robot.urdf (robot description, URDF)
Before this commit: robot diglobot2, 6 links, 5 joints
Links:
- added link gps_link; visual cylinder length=0.02 radius=0.025
Joints:
- added joint gps_joint: type fixed, parent base_footprint, child gps_link, origin xyz=-0.2 -0.0 0.3 rpy=0 0 0
